File: hardware/shield_v08/wat.sch (KiCad schematic (older format))
At the start: 38 parts, among them P101 24VOL, P102 CAUDAL_1, P103 V_IN, P104 PRESION_1, P105 INTENSIDAD_1, P106 18b20, P107 INTENSIDAD_2, P108 15VOL, P109 LCD_I2C, P110 ARD_DI_06, P111 ARD_ALI_04, P112 ARD_AN_04, P113 ARD_I2C_02, U101 ESP-12, U102 Recom-rd, U103 RO-1224S, U104 LM1117, U105 mp-1584, U106 NANO

Commit message: Add files via upload
Parts:
- removed D104: D, Diodes_ThroughHole:Diode_DO-35_SOD27_Horizontal_RM10, symbol D
- removed P108: 15VOL, Connect:bornier2, symbol CONN_01X02
- added D1: 1N4007, symbol D_ALT
- added D2: Schotky, symbol D_Schottky_Small_ALT
- added P108: 15VOL, Connect:bornier3, symbol CONN_01X03
- added TP1: 12v, symbol TEST
- added TP2: 8v, symbol TEST
- added TP3: 3v3, symbol TEST
- added TP4: 5v, symbol TEST
- C106, C107: value 22uF -> 100uF
- F101: value Fuse -> 2A
Connections:
- net labels added: Caudal_1, ESP_rst, ESP_rx, ESP_tx, Intensidad_1, Intensidad_2, Presión_1
- net labels removed: c_1, e_rst, e_rx, e_tx, i_1, i_2, p_1
- wire segments 110 -> 108
Other:
- note added: "+-15v"
- note added: "+24v"
- note added: "+3,3v"
- note added: "+8v"
- moved on the sheet: P112, P113, U102
