File: hardware/shield_v08/wat.sch (KiCad schematic (older format))
At the start: 37 parts, among them P101 24VOL, P102 CAUDAL_1, P103 V_IN, P104 PRESION_1, P105 INTENSIDAD_1, P106 18b20, P107 INTENSIDAD_2, P108 15VOL, P109 LCD_I2C, P110 ARD_DI_06, P111 ARD_ALI_04, U101 ESP-12, U102 Recom-rd, U103 RO-1224S, U104 LM1117, U105 mp-1584, U106 NANO

Commit message: [pdb] cambio posicion nano
Parts:
- added W101: +12V, Wire_Pads:SolderWirePad_single_0-8mmDrill, symbol TEST_1P
- added W102: +3,3V, Wire_Pads:SolderWirePad_single_0-8mmDrill, symbol TEST_1P
- added W103: +8V, Wire_Pads:SolderWirePad_single_0-8mmDrill, symbol TEST_1P
- D104: value D -> 1N4007
- P112: renamed from P?; footprint (none) -> Pin_Headers:Pin_Header_Straight_1x06
Connections:
- net labels added: caudal_1, intensidad_1, intensidad_2, presion_1
- net labels removed: c_1, i_1, i_2, p_1
- wire segments 110 -> 108

Commit message: [pcb]avance version 3
Parts:
- added D105: 1N4007, Diodes_ThroughHole:Diode_DO-35_SOD27_Horizontal_RM10, symbol D
- added P113: CONN_02X02, Pin_Headers:Pin_Header_Straight_2x02, symbol CONN_02X02
Connections:
- wire segments 108 -> 110
Other:
- moved on the sheet: C101, C102, C103, C104, D101, D102, D103, P102, P104, P105, P107, R101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
