File: hardware/shield_v08/_saved_wat.sch (KiCad schematic (older format))
At the start: 37 parts, among them P101 24VOL, P102 CAUDAL_1, P103 V_IN, P104 PRESION_1, P105 INTENSIDAD_1, P106 18b20, P107 INTENSIDAD_2, P108 15VOL, P109 LCD_I2C, P110 ARD_DI_06, P111 ARD_ALI_04, U101 ESP-12, U102 Recom-rd, U103 RO-1224S, U104 LM1117, U105 mp-1584, U106 NANO

Commit message: [pcb]mejoras version 3
Parts:
- P112: renamed from P?; value ARD_AN_I2C -> ARD_AN_I2C_06; footprint (none) -> Pin_Headers:Pin_Header_Straight_1x06
Changed lines of the file:
@@
 Connection ~ 1975 4625
 $Comp
-L CONN_01X06 P?
+L CONN_01X06 P112
 U 1 1 58AABC76
 P 6925 1950
-F 0 "P?" H 6925 2300 50  0000 C CNN
-F 1 "ARD_AN_I2C" V 7025 1950 50  0000 C CNN
-F 2 "" H 6925 1950 50  0000 C CNN
+F 0 "P112" H 6925 2300 50  0000 C CNN
+F 1 "ARD_AN_I2C_06" V 7025 1950 50  0000 C CNN
+F 2 "Pin_Headers:Pin_Header_Straight_1x06" H 6925 1950 50  0001 C CNN
 F 3 "" H 6925 1950 50  0000 C CNN
 	1    6925 1950

Commit message: [pcb]repongo librerias de huellas
Parts:
- P112: value ARD_AN_I2C_06 -> ARD_AN_I2C
Changed lines of the file:
@@
 P 6925 1950
 F 0 "P112" H 6925 2300 50  0000 C CNN
-F 1 "ARD_AN_I2C_06" V 7025 1950 50  0000 C CNN
+F 1 "ARD_AN_I2C" V 7025 1950 50  0000 C CNN
 F 2 "Pin_Headers:Pin_Header_Straight_1x06" H 6925 1950 50  0001 C CNN
 F 3 "" H 6925 1950 50  0000 C CNN

Commit message: [pdb] cambio posicion nano
Parts:
- added W101: +12V, Wire_Pads:SolderWirePad_single_0-8mmDrill, symbol TEST_1P
- added W102: +3,3V, Wire_Pads:SolderWirePad_single_0-8mmDrill, symbol TEST_1P
- added W103: +8V, Wire_Pads:SolderWirePad_single_0-8mmDrill, symbol TEST_1P
- D104: value D -> 1N4007
Connections:
- net labels added: caudal_1, intensidad_1, intensidad_2, presion_1
- net labels removed: c_1, i_1, i_2, p_1
- wire segments 110 -> 108
