File: hardware/shield_v09/wat.kicad_pcb (KiCad board)
At the start: 2 copper layers, 101 x 85.1 mm, 41 parts, among them P101 24VOL, P102 CAUDAL_1, P103 V_IN, P104 PRESION_1, P105 INTENSIDAD_1, P106 18b20, P107 INTENSIDAD_2, P108 15VOL, P109 LCD_I2C, P110 ARD_DI_06, P111 ARD_ALI_04, P112 ARD_AN_I2C, P113 CONN_02X02, U101 ESP-12, U102 Recom-rd, U103 RO-1224S, U104 LM1117, U105 mp-1584

Commit message: [pcb]version 3 completa
Parts:
- F101: footprint Fuse_Holders_and_Fuses:BladeFuse-Mini -> Fuse_Holders_and_Fuses:Fuseholder_Fuse_TR5_Littlefuse-No560_No460
- moved C105 10.5 mm to (138.0, 99.4), turned to 270 degrees
- moved U105 4.20 mm to (139.3, 115.0), turned to 90 degrees
- moved C101 3.78 mm to (60.5, 114.2)
- moved F101 3.76 mm to (134.5, 48.8)
- moved C102 2.50 mm to (76.3, 111.7)
- moved C103 2.50 mm to (86.3, 111.8)
- moved D102 2.50 mm to (78.3, 97.0)
- moved D103 2.50 mm to (88.8, 97.0)
- moved R102 2.50 mm to (72.7, 96.9)
- moved R103 2.50 mm to (82.3, 97.0)
- moved D104 2.25 mm to (142.0, 54.8)
- moved R101 1.88 mm to (60.5, 95.2)
- moved D101 1.65 mm to (65.8, 95.2)
Routing:
- net /Vin_12V: track 121.7 -> 150.4 mm
- net /Var_8V: track 174.4 -> 157.9 mm, vias 2 -> 0
- net /intensidad_2: track 64.5 -> 60.7 mm
- net /presion_1: track 56.7 -> 60.1 mm
- net Net-(F101-Pad1): track 9.24 -> 11.6 mm
- net Net-(C101-Pad1): track 14.8 -> 13.1 mm
- net Net-(C102-Pad1): track 15.1 -> 16.5 mm
- net Net-(C103-Pad1): track 15.1 -> 16.1 mm
