File: hardware/shield_v09/wat.sch (KiCad schematic (older format))
At the start: 43 parts, among them P101 24VOL, P102 CAUDAL_1, P103 V_IN, P104 PRESION_1, P105 INTENSIDAD_1, P106 18b20, P107 INTENSIDAD_2, P108 15VOL, P109 LCD_I2C, P110 ARD_DI_06, P111 ARD_ALI_04, P112 ARD_AN_I2C, P113 CONN_02X02, U101 ESP-12, U102 Recom-rd, U103 RO-1224S, U104 LM1117, U105 mp-1584, U106 NANO

Commit message: [pcb]version 3 completa
Parts:
- removed SHIELD?: ARDUINO_MEGA_SHIELD, symbol ARDUINO_MEGA_SHIELD
- F101: footprint Fuse_Holders_and_Fuses:BladeFuse-Mini -> Fuse_Holders_and_Fuses:Fuseholder_Fuse_TR5_Littlefuse-No560_No460
Connections:
- no-connect marks 126 -> 44
Changed lines of the file:
@@
 F 0 "F101" H 1310 1835 50  0000 L CNN
 F 1 "Fuse" H 1230 1715 50  0000 L CNN
-F 2 "Fuse_Holders_and_Fuses:BladeFuse-Mini" H 1350 1775 50  0001 C CNN
+F 2 "Fuse_Holders_and_Fuses:Fuseholder_Fuse_TR5_Littlefuse-No560_No460" H 1350 1775 50  0001 C CNN
 F 3 "" H 1350 1775 50  0000 C CNN
 	1    1350 1775
@@
 Text Label 3950 1500 0    60   ~ 0
 caudal_1
-$Comp
-L ARDUINO_MEGA_SHIELD SHIELD?
-U 1 1 58B0A291
-P 13700 2850
-F 0 "SHIELD?" H 13300 5350 60  0000 C CNN
-F 1 "ARDUINO_MEGA_SHIELD" H 13600 150 60  0000 C CNN
-F 2 "" H 13700 2850 60  0000 C CNN
-F 3 "" H 13700 2850 60  0000 C CNN
-	1    13700 2850
-	1    0    0    -1
-$EndComp
-NoConn ~ 14600 500
-NoConn ~ 14600 600
-NoConn ~ 14600 700
-NoConn ~ 14600 800
-NoConn ~ 14600 900
-NoConn ~ 14600 1000
-NoConn ~ 14600 1100
-NoConn ~ 14600 1200
-NoConn ~ 14600 1400
-NoConn ~ 14600 1500
-NoConn ~ 14600 1600
-NoConn ~ 14600 1700
-NoConn ~ 14600 1800
-NoConn ~ 14600 1900
-NoConn ~ 14600 2000
-NoConn ~ 14600 2100
-NoConn ~ 14600 2300
-NoConn ~ 14600 2400
-NoConn ~ 14600 2500
-NoConn ~ 14600 2600
-NoConn ~ 14600 2700
-NoConn ~ 14600 2800
-NoConn ~ 14600 2900
-NoConn ~ 14600 3000
-NoConn ~ 14600 3250
-NoConn ~ 14600 3350
-NoConn ~ 14600 3500
-NoConn ~ 14600 3600
-NoConn ~ 14600 3700
-NoConn ~ 14600 3800
-NoConn ~ 14600 3900
-NoConn ~ 14600 4000
-NoConn ~ 14600 4100
-NoConn ~ 14600 4200
-NoConn ~ 14600 4350
-NoConn ~ 14600 4450
-NoConn ~ 14600 4550
-NoConn ~ 14600 4650
-NoConn ~ 14600 4750
-NoConn ~ 14600 4850
-NoConn ~ 14600 4950
-NoConn ~ 14600 5050
-NoConn ~ 12700 900
-NoConn ~ 12700 1000
-NoConn ~ 12700 1100
-NoConn ~ 12700 1200
-NoConn ~ 12700 1300
-NoConn ~ 12700 1400
-NoConn ~ 12700 1600
-NoConn ~ 12700 1700
-NoConn ~ 12700 1800
-NoConn ~ 12700 1900
-NoConn ~ 12700 2000
-NoConn ~ 12700 2100
-NoConn ~ 12700 2200
-NoConn ~ 12700 2300
-NoConn ~ 12700 2500
-NoConn ~ 12700 2600
-NoConn ~ 12700 2700
-NoConn ~ 12700 2800
-NoConn ~ 12700 2900
-NoConn ~ 12700 3000
-NoConn ~ 12700 3100
-NoConn ~ 12700 3200
-NoConn ~ 12700 3700
-NoConn ~ 12700 3800
-NoConn ~ 12700 3900
-NoConn ~ 12700 4000
-NoConn ~ 12700 4150
-NoConn ~ 12700 4250
-NoConn ~ 12700 4350
-NoConn ~ 12700 4450
-NoConn ~ 12700 4550
-NoConn ~ 12700 4650
-NoConn ~ 12700 4750
-NoConn ~ 12700 4850
-NoConn ~ 12700 5000
-NoConn ~ 12700 5100
-NoConn ~ 12700 5200
-NoConn ~ 12700 5300
-NoConn ~ 12700 3450
-NoConn ~ 12700 3550
 $EndSCHEMATC
