File: hardware/shield_v10/wat.kicad_pcb (KiCad board)
At the start: 2 copper layers, 41 parts, among them P101 INTEN_1_V, P102 CAUDAL_1, P103 V_IN, P104 INTEN_1_I, P105 PRESION_1, P106 18b20, P107 INTEN_2_V, P108 INTEN_2_I, P109 LCD_I2C, P110 ARD_DI_06, P111 ARD_ALI_04, P112 ARD_AN_I2C, U101 ESP-12, U102 Recom-rd, U103 RO-1224S, U104 LM1117, U105 mp-1584

Commit message: [pcb] beta de la pcb
Parts:
- moved W103 18.1 mm to (175.0, 72.1)
- moved C102 9.63 mm to (139.3, 109.8)
- moved D102 9.22 mm to (124.0, 109.8)
- moved R105 8.45 mm to (131.3, 64.7), turned to 90 degrees
- moved R102 8.35 mm to (124.3, 105.6)
- moved C109 4.91 mm to (93.2, 62.1)
- moved U104 4.55 mm to (99.1, 59.7)
- moved C103 4.40 mm to (159.3, 109.8)
- moved D103 4.40 mm to (144.4, 109.8)
- moved W102 3.20 mm to (101.0, 67.5)
- moved R106 2.63 mm to (104.8, 66.6)
- moved C108 2.60 mm to (108.1, 71.1), turned to 180 degrees
- moved C106 2.40 mm to (101.9, 71.8)
- moved R103 1.90 mm to (144.4, 105.4)
- moved C107 0.69 mm to (155.9, 83.0)
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Connections:
- P110 pad 4: /e_tx -> /e_rx
- P110 pad 5: /e_rx -> /e_tx
Routing:
- net /Var_8V: track 0.00 -> 121.7 mm
- net /-15_voltios: track 0.00 -> 94.4 mm, vias 0 -> 2
- net /+15_voltios: track 0.00 -> 88.2 mm, vias 0 -> 2
- net /Vpc_5V: track 0.00 -> 87.0 mm, vias 0 -> 2
- net /caudal_1: track 0.00 -> 77.2 mm
- net /Vin_12V: track 0.00 -> 66.8 mm
- net /18b20: track 0.00 -> 57.4 mm
- net /presion_1: track 0.00 -> 54.4 mm
- net /e_tx: track 0.00 -> 35.5 mm
- net Net-(C102-Pad1): track 0.00 -> 35.1 mm
- net /intensidad_2: track 0.00 -> 33.8 mm
- net /e_rst: track 0.00 -> 33.4 mm
- net /Ves_3V3: track 0.00 -> 32.8 mm
- net /e_rx: track 0.00 -> 31.9 mm
- net /+24_voltios: track 0.00 -> 31.4 mm
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Other:
- board outline added: 101.8 x 85.9 mm

Commit message: [pcb] mejoras menores
Routing:
- net /Vpc_5V: track 87.0 -> 92.1 mm
- net /Ves_3V3: track 32.8 -> 34.6 mm
Changed lines of the file:
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@@
     (links 78)
     (no_connects 0)
-    (area 88.524999 43.524999 190.475001 129.575001)
+    (area 74.539287 31.545903 265.735715 296.250001)
     (thickness 1.6)
     (drawings 17)
-    (tracks 195)
+    (tracks 198)
     (zones 0)
     (modules 41)
@@
     (31 B.Cu signal)
     (32 B.Adhes user)
-    (33 F.Adhes user hide)
+    (33 F.Adhes user)
     (34 B.Paste user)
     (35 F.Paste user)
@@
   )
   (setup
-    (last_trace_width 0.8)
+    (last_trace_width 1)
     (user_trace_width 0.4)
     (user_trace_width 0.6)
@@
   (segment (start 184.319 73.681) (end 184.319 76.096) (width 1.2) (layer B.Cu) (net 18))
   (segment (start 185.49746 72.50254) (end 184.319 73.681) (width 1.2) (layer B.Cu) (net 18))
-  (segment (start 104.8 66.6) (end 108 69.8) (width 0.8) (layer B.Cu) (net 19))
-  (segment (start 108 69.8) (end 108 71) (width 0.8) (layer B.Cu) (net 19))
+  (segment (start 104.8 66.6) (end 105.1 66.6) (width 1) (layer B.Cu) (net 19))
+  (segment (start 105.1 66.6) (end 108.1 69.6) (width 1) (layer B.Cu) (net 19))
+  (segment (start 108.1 69.6) (end 108.1 71.1) (width 1) (layer B.Cu) (net 19))
+  (segment (start 104.8 66.6) (end 104.8 67.3) (width 1) (layer B.Cu) (net 19))
+  (segment (start 104.8 67.3) (end 101.9 70.2) (width 1) (layer B.Cu) (net 19))
+  (segment (start 101.9 70.2) (end 101.9 71.8) (width 1) (layer B.Cu) (net 19))
+  (segment (start 104.8 66.6) (end 110.65 66.6) (width 1) (layer B.Cu) (net 19))
+  (segment (start 110.65 66.6) (end 110.75 66.7) (width 1) (layer B.Cu) (net 19))
+  (segment (start 100.95 67.5) (end 100.95 67) (width 1) (layer B.Cu) (net 19))
+  (segment (start 100.95 67) (end 101.35 66.6) (width 1) (layer B.Cu) (net 19))
+  (segment (start 101.35 66.6) (end 104.8 66.6) (width 1) (layer B.Cu) (net 19))
+  (segment (start 99.1 59.7) (end 101.5 59.7) (width 1) (layer B.Cu) (net 19))
+  (segment (start 104.8 63) (end 104.8 66.6) (width 1) (layer B.Cu) (net 19))
+  (segment (start 101.5 59.7) (end 104.8 63) (width 1) (layer B.Cu) (net 19))
   (segment (start 108 71) (end 108.1 71.1) (width 0.8) (layer B.Cu) (net 19))
-  (segment (start 101.9 70.15) (end 101.9 71.8) (width 0.8) (layer B.Cu) (net 19))
-  (segment (start 104.8 67.25) (end 101.9 70.15) (width 0.8) (layer B.Cu) (net 19))
   (segment (start 104.8 66.6) (end 104.8 67.25) (width 0.8) (layer B.Cu) (net 19))
-  (segment (start 101.85 66.6) (end 100.95 67.5) (width 0.8) (layer B.Cu) (net 19))
-  (segment (start 104.8 66.6) (end 101.85 66.6) (width 0.8) (layer B.Cu) (net 19))
-  (segment (start 99.1 59.7) (end 100.9 59.7) (width 0.8) (layer B.Cu) (net 19))
-  (segment (start 104.8 63.6) (end 104.8 66.6) (width 0.8) (layer B.Cu) (net 19))
-  (segment (start 100.9 59.7) (end 104.8 63.6) (width 0.8) (layer B.Cu) (net 19))
-  (segment (start 104.8 66.6) (end 110.65 66.6) (width 0.8) (layer B.Cu) (net 19))
   (segment (start 110.65 66.6) (end 110.75 66.7) (width 0.8) (layer B.Cu) (net 19))
   (segment (start 175 72.1) (end 165.7 76.019) (width 0.8) (layer B.Cu) (net 20) (status 10))
@@
   (segment (start 96.95 67.25) (end 96.95 79.5) (width 1.2) (layer B.Cu) (net 20))
   (segment (start 99.1 65.1) (end 96.95 67.25) (width 1.2) (layer B.Cu) (net 20))
-  (segment (start 123.15 98.2) (end 122.75 98.2) (width 0.8) (layer B.Cu) (net 21))
-  (segment (start 122.75 98.2) (end 121.3225 96.7725) (width 0.8) (layer B.Cu) (net 21))
+  (segment (start 121.3225 96.5275) (end 121.3775 96.5275) (width 1) (layer B.Cu) (net 21))
+  (segment (start 145.35 65.1) (end 156.53948 65.1) (width 1) (layer B.Cu) (net 21))
+  (segment (start 139.1 71.35) (end 145.35 65.1) (width 1) (layer B.Cu) (net 21))
+  (via (at 139.1 71.35) (size 0.6) (drill 0.4) (layers F.Cu B.Cu) (net 21))
+  (segment (start 139.1 87.5) (end 139.1 71.35) (width 1) (layer F.Cu) (net 21))
+  (segment (start 139.05 87.55) (end 139.1 87.5) (width 1) (layer F.Cu) (net 21))
+  (via (at 139.05 87.55) (size 0.6) (drill 0.4) (layers F.Cu B.Cu) (net 21))
+  (segment (start 139.05 91.85) (end 139.05 87.55) (width 1) (layer B.Cu) (net 21))
+  (segment (start 132.8 98.1) (end 139.05 91.85) (width 1) (layer B.Cu) (net 21))
+  (segment (start 122.95 98.1) (end 132.8 98.1) (width 1) (layer B.Cu) (net 21))
+  (segment (start 121.3775 96.5275) (end 122.95 98.1) (width 1) (layer B.Cu) (net 21))
+  (segment (start 121.3225 95.1825) (end 121.3225 96.5275) (width 1) (layer B.Cu) (net 21))
+  (segment (start 116.305 101.545) (end 116.305 102.85) (width 1) (layer B.Cu) (net 21))
+  (segment (start 121.3225 96.5275) (end 116.305 101.545) (width 1) (layer B.Cu) (net 21))
   (segment (start 156.53948 68.62754) (end 156.53948 68.66052) (width 0.8) (layer B.Cu) (net 21))
-  (segment (start 156.53948 68.66052) (end 154.5 70.7) (width 0.8) (layer B.Cu) (net 21))
-  (segment (start 136.55 98.2) (end 123.15 98.2) (width 0.8) (layer B.Cu) (net 21))
-  (segment (start 123.15 98.2) (end 123 98.2) (width 0.8) (layer B.Cu) (net 21))
-  (segment (start 148.55 86.2) (end 136.55 98.2) (width 0.8) (layer B.Cu) (net 21))
-  (via (at 148.55 86.2) (size 1.9) (drill 1) (layers F.Cu B.Cu) (net 21))
-  (segment (start 148.55 72.15) (end 148.55 86.2) (width 0.8) (layer F.Cu) (net 21))
-  (via (at 148.55 72.15) (size 1.9) (drill 1) (layers F.Cu B.Cu) (net 21))
-  (segment (start 148.55 72.1) (end 148.55 72.15) (width 0.8) (layer B.Cu) (net 21))
-  (segment (start 149.95 70.7) (end 148.55 72.1) (width 0.8) (layer B.Cu) (net 21))
-  (segment (start 154.5 70.7) (end 149.95 70.7) (width 0.8) (layer B.Cu) (net 21))
-  (segment (start 156.53948 68.62754) (end 156.53948 64.81052) (width 1) (layer B.Cu) (net 21))
+  (segment (start 156.53948 68.62754) (end 156.53948 65.1) (width 1) (layer B.Cu) (net 21))
+  (segment (start 156.53948 65.1) (end 156.53948 64.81052) (width 1) (layer B.Cu) (net 21))
+  (segment (start 156.53948 64.81052) (end 159.585 61.765) (width 1) (layer B.Cu) (net 21))
   (segment (start 159.585 61.765) (end 159.585 58.625) (width 1) (layer B.Cu) (net 21))
-  (segment (start 156.53948 64.81052) (end 159.585 61.765) (width 1) (layer B.Cu) (net 21))
   (segment (start 160.58 49.525) (end 160.58 53.42) (width 1) (layer B.Cu) (net 21))
   (segment (start 160.58 53.42) (end 159.585 54.415) (width 1) (layer B.Cu) (net 21))
   (segment (start 159.585 54.415) (end 159.585 58.625) (width 1) (layer B.Cu) (net 21))
-  (segment (start 121.3225 95.1825) (end 121.3225 96.7725) (width 1) (layer B.Cu) (net 21))
-  (segment (start 121.3225 96.7725) (end 121.3225 96.7775) (width 1) (layer B.Cu) (net 21))
-  (segment (start 121.3225 96.7775) (end 116.305 101.795) (width 1) (layer B.Cu) (net 21))
-  (segment (start 116.305 101.795) (end 116.305 102.85) (width 1) (layer B.Cu) (net 21))
   (segment (start 155.5 49.525) (end 155.5 53) (width 0.8) (layer B.Cu) (net 22))
   (segment (start 155.5 53) (end 149.875 58.625) (width 0.8) (layer B.Cu) (net 22))

Commit message: [hardware]v10 y pinza
Parts:
- R101, R102, R103: footprint Resistors_ThroughHole:Resistor_Horizontal_RM15mm -> oscar_libreria_huellas:Resistor_RM15mm_pad
- U101: footprint ESP8266:ESP-07v2 -> oscar_libreria_huellas:ESP-07v2_pad
- moved C107 3.05 mm to (155.9, 86.1)
- moved R102 0.41 mm to (124.7, 105.5)
- moved C102 0.35 mm to (139.7, 109.8)
- moved R101 0.28 mm to (93.1, 109.7)
Routing:
- net /Var_8V: track 121.7 -> 125.9 mm
