File: hardware/shield_v10/wat.sch (KiCad schematic (older format))
At the start: 42 parts, among them P101 INTEN_1_V, P102 CAUDAL_1, P103 V_IN, P104 INTEN_1_I, P105 PRESION_1, P106 18b20, P107 INTEN_2_V, P108 INTEN_2_I, P109 LCD_I2C, P110 ARD_DI_06, P111 ARD_ALI_04, P112 ARD_AN_I2C, U101 ESP-12, U102 Recom-rd, U103 RO-1224S, U104 LM1117, U105 mp-1584, U106 NANO

Commit message: [pcb] beta de la pcb
Changed lines of the file:
@@
 	1    0    0    -1
 $EndComp
-Text Label 4325 1900 2    60   ~ 0
+Text Label 4350 1800 2    60   ~ 0
 e_rx
-Text Label 4325 1800 2    60   ~ 0
+Text Label 4350 1900 2    60   ~ 0
 e_tx
 Text Label 4375 2000 2    60   ~ 0
@@
 	2700 5375 2700 5525
 Wire Wire Line
-	2600 5275 2800 5275
-Wire Wire Line
-	2600 5475 2800 5475
-Wire Wire Line
 	875  4100 1050 4100
 Wire Wire Line
@@
 Wire Wire Line
 	10400 3100 10525 3100
-Text Label 2800 5275 0    60   ~ 0
-+15_voltios
-Text Label 2800 5475 0    60   ~ 0
--15_voltios
 Wire Wire Line
 	10525 2900 10225 2900
@@
 Wire Wire Line
 	10450 3925 9750 3925
-Text Label 9750 3925 0    60   ~ 0
-+15_voltios
-Text Label 9750 4075 0    60   ~ 0
--15_voltios
 Text Label 2800 6225 0    60   ~ 0
 +24_voltios
@@
 	1    0    0    1
 $EndComp
+Wire Wire Line
+	2600 5275 3000 5275
+Wire Wire Line
+	2600 5475 3000 5475
+Text Label 2775 5275 0    60   ~ 0
++15_voltios
+Text Label 2775 5475 0    60   ~ 0
+-15_voltios
+Text Label 9750 3925 0    60   ~ 0
++15_voltios
+Text Label 9750 4075 0    60   ~ 0
+-15_voltios
 $EndSCHEMATC

Commit message: [hardware]v10 y pinza
Parts:
- R101, R102, R103: footprint Resistors_ThroughHole:Resistor_Horizontal_RM15mm -> oscar_libreria_huellas:Resistor_RM15mm_pad
- U101: footprint ESP8266:ESP-07v2 -> oscar_libreria_huellas:ESP-07v2_pad
Changed lines of the file:
@@
 F 0 "U101" H 5725 3975 50  0000 C CNN
 F 1 "ESP-12" H 5725 4175 50  0000 C CNN
-F 2 "ESP8266:ESP-07v2" H 5725 4075 50  0001 C CNN
+F 2 "oscar_libreria_huellas:ESP-07v2_pad" H 5725 4075 50  0001 C CNN
 F 3 "" H 5725 4075 50  0001 C CNN
 	1    5725 4075
@@
 F 0 "R101" V 9880 3000 50  0000 C CNN
 F 1 "1K" V 9800 3000 50  0000 C CNN
-F 2 "Resistors_ThroughHole:Resistor_Horizontal_RM15mm" V 9730 3000 50  0001 C CNN
+F 2 "oscar_libreria_huellas:Resistor_RM15mm_pad" V 9730 3000 50  0001 C CNN
 F 3 "" H 9800 3000 50  0000 C CNN
 	1    9800 3000
@@
 F 0 "R102" V 9930 4350 50  0000 C CNN
 F 1 "1K" V 9850 4350 50  0000 C CNN
-F 2 "Resistors_ThroughHole:Resistor_Horizontal_RM15mm" V 9780 4350 50  0001 C CNN
+F 2 "oscar_libreria_huellas:Resistor_RM15mm_pad" V 9780 4350 50  0001 C CNN
 F 3 "" H 9850 4350 50  0000 C CNN
 	1    9850 4350
@@
 F 0 "R103" V 9930 5625 50  0000 C CNN
 F 1 "1K" V 9850 5625 50  0000 C CNN
-F 2 "Resistors_ThroughHole:Resistor_Horizontal_RM15mm" V 9780 5625 50  0001 C CNN
+F 2 "oscar_libreria_huellas:Resistor_RM15mm_pad" V 9780 5625 50  0001 C CNN
 F 3 "" H 9850 5625 50  0000 C CNN
 	1    9850 5625
