File: hardware/pinza/pinza.kicad_pcb (KiCad board)
At the start: 2 copper layers, 49 x 26.7 mm, 8 parts, among them P101 5V_ENTRADA, P102 PINZA, U101 NodeMCU_Amica_R2_0

Commit message: [hardware]pinza nodemcu
Parts:
- added C1: CP1, Capacitors_ThroughHole:C_Radial_D5_L11_P2, F.Cu at (135.9, 104.1)
- moved C101 3.41 mm to (120.7, 97.8)
Routing:
- net /3V3: track 7.57 -> 13.6 mm
- net Net-(C101-Pad1): track 42.6 -> 46.0 mm
Changed lines of the file:
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@@
 (kicad_pcb (version 4) (host pcbnew 4.0.2+dfsg1-stable)
   (general
-    (links 16)
+    (links 18)
     (no_connects 0)
     (area 98.395 71.901189 173.375 115.840001)
     (thickness 1.6)
     (drawings 4)
-    (tracks 22)
+    (tracks 24)
     (zones 0)
-    (modules 8)
+    (modules 9)
     (nets 29)
   )
@@
   )
   (setup
-    (last_trace_width 0.25)
+    (last_trace_width 1.2)
     (user_trace_width 0.6)
     (user_trace_width 0.8)
@@
     (visible_elements FFFFFF7F)
     (pcbplotparams
-      (layerselection 0x00030_80000001)
+      (layerselection 0x01030_80000001)
       (usegerberextensions false)
       (excludeedgelayer true)
@@
   )
   (module Capacitors_ThroughHole:C_Radial_D5_L11_P2 (layer F.Cu)
-    (at 120.8 101.2 90)
+    (at 120.65 97.79 90)
     (descr "Radial Electrolytic Capacitor 5mm x Length 11mm, Pitch 2mm")
     (tags "Electrolytic Capacitor")
@@
     )
   )
+  (module Capacitors_ThroughHole:C_Radial_D5_L11_P2 (layer F.Cu)
+    (at 135.89 104.14 90)
+    (descr "Radial Electrolytic Capacitor 5mm x Length 11mm, Pitch 2mm")
+    (tags "Electrolytic Capacitor")
+    (fp_text reference C1 (at 1 -3.8 90) (layer F.SilkS)
+      (effects (font (size 1 1) (thickness 0.15)))
+    )
+    (fp_text value CP1 (at 1 3.8 90) (layer F.Fab)
+      (effects (font (size 1 1) (thickness 0.15)))
+    )
+    (fp_line (start 1.075 -2.499) (end 1.075 2.499) (layer F.SilkS) (width 0.15))
+    (fp_line (start 1.215 -2.491) (end 1.215 -0.154) (layer F.SilkS) (width 0.15))
+    (fp_line (start 1.215 0.154) (end 1.215 2.491) (layer F.SilkS) (width 0.15))
+    (fp_line (start 1.355 -2.475) (end 1.355 -0.473) (layer F.SilkS) (width 0.15))
+    (fp_line (start 1.355 0.473) (end 1.355 2.475) (layer F.SilkS) (width 0.15))
+    (fp_line (start 1.495 -2.451) (end 1.495 -0.62) (layer F.SilkS) (width 0.15))
+    (fp_line (start 1.495 0.62) (end 1.495 2.451) (layer F.SilkS) (width 0.15))
+    (fp_line (start 1.635 -2.418) (end 1.635 -0.712) (layer F.SilkS) (width 0.15))
+    (fp_line (start 1.635 0.712) (end 1.635 2.418) (layer F.SilkS) (width 0.15))
+    (fp_line (start 1.775 -2.377) (end 1.775 -0.768) (layer F.SilkS) (width 0.15))
+    (fp_line (start 1.775 0.768) (end 1.775 2.377) (layer F.SilkS) (width 0.15))
+    (fp_line (start 1.915 -2.327) (end 1.915 -0.795) (layer F.SilkS) (width 0.15))
+    (fp_line (start 1.915 0.795) (end 1.915 2.327) (layer F.SilkS) (width 0.15))
+    (fp_line (start 2.055 -2.266) (end 2.055 -0.798) (layer F.SilkS) (width 0.15))
+    (fp_line (start 2.055 0.798) (end 2.055 2.266) (layer F.SilkS) (width 0.15))
+    (fp_line (start 2.195 -2.196) (end 2.195 -0.776) (layer F.SilkS) (width 0.15))
+    (fp_line (start 2.195 0.776) (end 2.195 2.196) (layer F.SilkS) (width 0.15))
+    (fp_line (start 2.335 -2.114) (end 2.335 -0.726) (layer F.SilkS) (width 0.15))
+    (fp_line (start 2.335 0.726) (end 2.335 2.114) (layer F.SilkS) (width 0.15))
+    (fp_line (start 2.475 -2.019) (end 2.475 -0.644) (layer F.SilkS) (width 0.15))
+    (fp_line (start 2.475 0.644) (end 2.475 2.019) (layer F.SilkS) (width 0.15))
+    (fp_line (start 2.615 -1.908) (end 2.615 -0.512) (layer F.SilkS) (width 0.15))
+    (fp_line (start 2.615 0.512) (end 2.615 1.908) (layer F.SilkS) (width 0.15))
+    (fp_line (start 2.755 -1.78) (end 2.755 -0.265) (layer F.SilkS) (width 0.15))
+    (fp_line (start 2.755 0.265) (end 2.755 1.78) (layer F.SilkS) (width 0.15))
+    (fp_line (start 2.895 -1.631) (end 2.895 1.631) (layer F.SilkS) (width 0.15))
+    (fp_line (start 3.035 -1.452) (end 3.035 1.452) (layer F.SilkS) (width 0.15))
+    (fp_line (start 3.175 -1.233) (end 3.175 1.233) (layer F.SilkS) (width 0.15))
+    (fp_line (start 3.315 -0.944) (end 3.315 0.944) (layer F.SilkS) (width 0.15))
+    (fp_line (start 3.455 -0.472) (end 3.455 0.472) (layer F.SilkS) (width 0.15))
+    (fp_circle (center 2 0) (end 2 -0.8) (layer F.SilkS) (width 0.15))
+    (fp_circle (center 1 0) (end 1 -2.5375) (layer F.SilkS) (width 0.15))
+    (fp_circle (center 1 0) (end 1 -2.8) (layer F.CrtYd) (width 0.05))
+    (pad 1 thru_hole rect (at 0 0 90) (size 1.3 1.3) (drill 0.8) (layers *.Cu *.Mask F.SilkS)
+      (net 5 /3V3))
+    (pad 2 thru_hole circle (at 2 0 90) (size 1.3 1.3) (drill 0.8) (layers *.Cu *.Mask F.SilkS)
+      (net 2 GND))
+    (model Capacitors_ThroughHole.3dshapes/C_Radial_D5_L11_P2.wrl
+      (at (xyz 0 0 0))
+      (scale (xyz 1 1 1))
+      (rotate (xyz 0 0 0))
+    )
+  )
   (gr_line (start 100.8 115.6) (end 100.8 88.9) (angle 90) (layer Edge.Cuts) (width 0.15))
   (gr_line (start 149.8 115.6) (end 100.8 115.6) (angle 90) (layer Edge.Cuts) (width 0.15))
   (gr_line (start 149.8 88.9) (end 149.8 115.6) (angle 90) (layer Edge.Cuts) (width 0.15))
   (gr_line (start 100.9 88.9) (end 149.8 88.9) (angle 90) (layer Edge.Cuts) (width 0.15))
+  (segment (start 120.65 97.79) (end 120.65 108.55) (width 1.2) (layer B.Cu) (net 1) (status C00000))
+  (segment (start 120.65 108.55) (end 120 109.2) (width 1.2) (layer B.Cu) (net 1) (status C00000))
   (segment (start 110.7 102.3) (end 105.46 102.3) (width 1.2) (layer B.Cu) (net 1))
   (segment (start 105.46 102.3) (end 104.6 101.44) (width 1.2) (layer B.Cu) (net 1))
@@
   (segment (start 114.9 105.3) (end 116 105.2) (width 1.2) (layer B.Cu) (net 1) (status 10))
   (segment (start 116 105.2) (end 120 109.2) (width 1.2) (layer B.Cu) (net 1))
-  (segment (start 120.8 101.2) (end 120.8 108.4) (width 1.2) (layer B.Cu) (net 1))
-  (segment (start 120.8 108.4) (end 120 109.2) (width 1.2) (layer B.Cu) (net 1))
   (segment (start 120 109.2) (end 128.34 109.2) (width 1.2) (layer B.Cu) (net 1))
   (segment (start 128.34 109.2) (end 128.54 109) (width 1.2) (layer B.Cu) (net 1))
@@
   (segment (start 107.2 90.8) (end 107.2 93.76) (width 1.2) (layer B.Cu) (net 4))
   (segment (start 107.2 93.76) (end 104.6 96.36) (width 1.2) (layer B.Cu) (net 4))
+  (segment (start 135.89 104.14) (end 135.89 106.19) (width 1.2) (layer B.Cu) (net 5) (status 400000))
+  (segment (start 135.89 106.19) (end 138.7 109) (width 1.2) (layer B.Cu) (net 5) (status 800000))
   (segment (start 138.7 109) (end 140.8 109) (width 1.2) (layer B.Cu) (net 5))
   (segment (start 142.76 110.96) (end 142.76 113.66) (width 1.2) (layer B.Cu) (net 5))
