File: hardware/pinza/pinza.sch (KiCad schematic (older format))
At the start: 8 parts, among them P101 5V_ENTRADA, P102 PINZA, U101 NodeMCU_Amica_R2_0

Commit message: [hardware]pinza nodemcu
Parts:
- added C1: CP1, Capacitors_ThroughHole:C_Radial_D5_L11_P2, symbol CP1
Connections:
- wire segments 22 -> 25
Changed lines of the file:
@@
 Connection ~ 6200 2375
 $Comp
-L GND #PWR?
+L GND #PWR010
 U 1 1 592B1964
 P 4000 1800
-F 0 "#PWR?" H 4000 1550 50  0001 C CNN
+F 0 "#PWR010" H 4000 1550 50  0001 C CNN
 F 1 "GND" H 4000 1650 50  0000 C CNN
 F 2 "" H 4000 1800 50  0000 C CNN
@@
 Wire Wire Line
 	3825 1800 4000 1800
+$Comp
+L CP1 C1
+U 1 1 5947CB6B
+P 4805 1675
+F 0 "C1" H 4830 1775 50  0000 L CNN
+F 1 "CP1" H 4830 1575 50  0000 L CNN
+F 2 "Capacitors_ThroughHole:C_Radial_D5_L11_P2" H 4805 1675 50  0001 C CNN
+F 3 "" H 4805 1675 50  0000 C CNN
+	1    4805 1675
+	1    0    0    -1
+$EndComp
+Wire Wire Line
+	4805 1525 4805 1420
+Wire Wire Line
+	4805 1420 5175 1420
+Connection ~ 5175 1420
+$Comp
+L GND #PWR011
+U 1 1 5947CCC7
+P 4805 1890
+F 0 "#PWR011" H 4805 1640 50  0001 C CNN
+F 1 "GND" H 4805 1740 50  0000 C CNN
+F 2 "" H 4805 1890 50  0000 C CNN
+F 3 "" H 4805 1890 50  0000 C CNN
+	1    4805 1890
+	1    0    0    -1
+$EndComp
+Wire Wire Line
+	4805 1825 4805 1890
 $EndSCHEMATC
